Commit message: code

File: urdf/sherlock_robot.xacro (robot description, xacro)
@@ -1,7 +1,7 @@
 <?xml version="1.0"?>
-<robot xmlns:xacro="http://www.ros.org/wiki/xacro" name="sherlock_robot_xacro">
+<robot xmlns:xacro="http://www.ros.org/wiki/xacro" name="sherlock robot">
 <xacro:include filename="$(find erl_assignment3)/urdf/sherlock_robot.gazebo"/>
-	<xacro:property name="length_wheel" value="0.02" />
-	<xacro:property name="radius_wheel" value="0.05" />
+	<xacro:property name="length_wheel" value="0.04" />
+	<xacro:property name="radius_wheel" value="0.1" />
 	<xacro:macro name="default_inertial" params="mass">
                <inertial>
@@ -51,11 +51,11 @@
     <collision name="collision_chassis">
       <geometry>
-        <box size="0.25 0.15 0.035"/>
+        <box size="0.5 0.3 0.07"/>
       </geometry>
     </collision>
     <visual>
-      <origin rpy="0 0 0" xyz="0 0 0"/>
-      <geometry>
-        <box size="0.25 0.15 0.035"/>
+      <origin rpy="0 0 0" xyz="0 0 0.0"/>
+      <geometry>
+        <box size="0.5 0.3 0.07"/>
       </geometry>
       <material name="blue"/>
@@ -63,13 +63,13 @@
     <!-- caster front -->
     <collision name="caster_front_collision">
-      <origin rpy=" 0 0 0" xyz="0.175 0 -0.025"/>
-      <geometry>
-        <sphere radius="0.025"/>
+      <origin rpy=" 0 0 0" xyz="0.35 0 -0.05"/>
+      <geometry>
+        <sphere radius="0.05"/>
       </geometry>
     </collision>
     <visual name="caster_front_visual">
-      <origin rpy=" 0 0 0" xyz="0.1 0 -0.025"/>
-      <geometry>
-        <sphere radius="0.025"/>
+      <origin rpy=" 0 0 0" xyz="0.2 0 -0.05"/>
+      <geometry>
+        <sphere radius="0.05"/>
       </geometry>
     </visual>
@@ -100,5 +100,5 @@
   </link>
   <joint name="joint_right_wheel" type="continuous">
-    <origin rpy="0 0 0" xyz="-0.025 0.075 0"/>
+    <origin rpy="0 0 0" xyz="-0.05 0.15 0"/>
     <child link="link_right_wheel"/>
     <parent link="link_chassis"/>
@@ -108,5 +108,5 @@
   </joint>
   <joint name="joint_left_wheel" type="continuous">
-    <origin rpy="0 0 0" xyz="-0.025 -0.075 0"/>
+    <origin rpy="0 0 0" xyz="-0.05 -0.15 0"/>
     <child link="link_left_wheel"/>
     <parent link="link_chassis"/>
@@ -117,13 +117,13 @@
   <link name="hokuyo_link">
 	    <collision>
-	      <origin xyz="0 0 0.00125" rpy="0 0 0"/>
-	      <geometry>
-		<box size="0.025 0.025 0.025"/>
+	      <origin xyz="0 0 0.025" rpy="0 0 0"/>
+	      <geometry>
+		<box size="0.05 0.05 0.05"/>
 	      </geometry>
 	    </collision>
 	    <visual>
-	      <origin xyz="0 0 0.0125" rpy="0 0 0"/>
-	      <geometry>
-		<box size="0.025 0.025 0.025"/>
+	      <origin xyz="0 0 0.025" rpy="0 0 0"/>
+	      <geometry>
+		<box size="0.05 0.05 0.05"/>
 	      </geometry>
 	      <material name="red">
@@ -139,7 +139,63 @@
   <joint name="hokuyo_joint" type="fixed">
 	    <axis xyz="0 1 0" />
-	    <origin xyz="0.14 0 0.025" rpy="0 0 0"/>
+	    <origin xyz="0.28 0 0.05" rpy="0 0 0"/>
 	    <parent link="link_chassis"/>
 	    <child link="hokuyo_link"/>
 	 </joint>
+  <link name="camera_link">
+	    <collision>
+	      <origin xyz="0 0 0.5" rpy="0 0 0"/>
+	      <geometry>
+		<box size="0.05 0.05 0.05"/>
+	      </geometry>
+	    </collision>
+	    <visual>
+	      <origin xyz="0 0 0.5" rpy="0 0 0"/>
+	      <geometry>
+		<box size="0.05 0.05 0.05"/>
+	      </geometry>
+	      <material name="red">
+		<color rgba="1 0 0 1"/>
+	      </material>
+	    </visual>
+	    <inertial>
+	      <mass value="1e-5" />
+	      <origin xyz="0 0 0.5" rpy="0 0 0"/>
+	      <inertia ixx="1e-6" ixy="0" ixz="0" iyy="1e-6" iyz="0" izz="1e-6" />
+	    </inertial>
+  </link>
+  <joint name="camera_joint" type="fixed">
+	    <axis xyz="0 1 0" />
+	    <origin xyz="0.6 0 0.5" rpy="0 0 0"/>
+	    <parent link="link_chassis"/>
+	    <child link="camera_link"/>
+ </joint>
+ <link name="camera_floor_link">
+	    <collision>
+	      <origin xyz="0.0 0 0.8" rpy="0 1.57 0"/>
+	      <geometry>
+		<box size="0.05 0.05 0.05"/>
+	      </geometry>
+	    </collision>
+	    <visual>
+	      <origin xyz="0.0 0 0.8" rpy="0 1.57 0"/>
+	      <geometry>
+		<box size="0.05 0.05 0.05"/>
+	      </geometry>
+	      <material name="red">
+		<color rgba="1 0 0 1"/>
+	      </material>
+	    </visual>
+	    <inertial>
+	      <mass value="1e-5" />
+	      <origin xyz="0.0 0 0.8" rpy="0 1.57 0"/>
+	      <inertia ixx="1e-6" ixy="0" ixz="0" iyy="1e-6" iyz="0" izz="1e-6" />
+	    </inertial>
+  </link>
+  <joint name="camera_floor_joint" type="fixed">
+	    <axis xyz="0 1 0" />
+	    <origin xyz="0.8 0 0.8" rpy="0 1.57 0"/>
+	    <parent link="link_chassis"/>
+	    <child link="camera_floor_link"/>
+ </joint>
 </robot>
